File: hardware/Weather Station Motherboard V1/Weather Station Motherboard V1.kicad_sch (KiCad schematic)
At the start: 33 parts, among them J1 Conn_01x02, J2 Conn_02x03_Odd_Even, J3 Conn_01x04, U1 ESP32-WROOM-32, U2 SHTC3, U3 BMP390, U4 TPS62177DQC

Commit message: Added jumpers
Added jumper connections to seperate pressure sensors unless soldered together
Parts:
- added JP1: SolderJumper_2_Open, Jumper:SolderJumper-2_P1.3mm_Open_RoundedPad1.0x1.5mm, symbol Jumper:SolderJumper_2_Open
- added JP2, JP3, JP4: SolderJumper_2_Open, Jumper:SolderJumper-2_P1.3mm_Open_Pad1.0x1.5mm, symbol Jumper:SolderJumper_2_Open
Changed lines of the file:
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@@
+    )
+  )
+  (symbol (lib_id "Jumper:SolderJumper_2_Open") (at 190.5 80.01 0) (unit 1)
+    (in_bom yes) (on_board yes) (dnp no) (fields_autoplaced)
+    (property "Reference" "JP4" (at 190.5 73.66 0)
+      (effects (font (size 1.27 1.27)))
+    )
+    (property "Value" "SolderJumper_2_Open" (at 190.5 76.2 0)
+      (effects (font (size 1.27 1.27)))
+    )
+    (property "Footprint" "Jumper:SolderJumper-2_P1.3mm_Open_Pad1.0x1.5mm" (at 190.5 80.01 0)
+      (effects (font (size 1.27 1.27)) hide)
+    )
+    (property "Datasheet" "~" (at 190.5 80.01 0)
+      (effects (font (size 1.27 1.27)) hide)
+    )
+    (pin "1")
+    (pin "2")
+    (instances
+      (project "Weather Station Motherboard V1"
+        (path "/782b25c2-8b22-49ba-9398-f7481b8d9716"
+          (reference "JP4") (unit 1)
+        )
+      )
     )
   )
@@
         (path "/782b25c2-8b22-49ba-9398-f7481b8d9716"
           (reference "U5") (unit 1)
+        )
+      )
+    )
+  )
+  (symbol (lib_id "Jumper:SolderJumper_2_Open") (at 190.5 102.87 0) (unit 1)
+    (in_bom yes) (on_board yes) (dnp no) (fields_autoplaced)
+    (property "Reference" "JP2" (at 190.5 96.52 0)
+      (effects (font (size 1.27 1.27)))
+    )
+    (property "Value" "SolderJumper_2_Open" (at 190.5 99.06 0)
+      (effects (font (size 1.27 1.27)))
+    )
+    (property "Footprint" "Jumper:SolderJumper-2_P1.3mm_Open_Pad1.0x1.5mm" (at 190.5 102.87 0)
+      (effects (font (size 1.27 1.27)) hide)
+    )
+    (property "Datasheet" "~" (at 190.5 102.87 0)
+      (effects (font (size 1.27 1.27)) hide)
+    )
+    (pin "1")
+    (pin "2")
+    (instances
+      (project "Weather Station Motherboard V1"
+        (path "/782b25c2-8b22-49ba-9398-f7481b8d9716"
+          (reference "JP2") (unit 1)
         )
       )
@@
     )
   )
+  (symbol (lib_id "Jumper:SolderJumper_2_Open") (at 190.5 93.98 0) (unit 1)
+    (in_bom yes) (on_board yes) (dnp no) (fields_autoplaced)
+    (property "Reference" "JP3" (at 190.5 87.63 0)
+      (effects (font (size 1.27 1.27)))
+    )
+    (property "Value" "SolderJumper_2_Open" (at 190.5 90.17 0)
+      (effects (font (size 1.27 1.27)))
+    )
+    (property "Footprint" "Jumper:SolderJumper-2_P1.3mm_Open_Pad1.0x1.5mm" (at 190.5 93.98 0)
+      (effects (font (size 1.27 1.27)) hide)
+    )
+    (property "Datasheet" "~" (at 190.5 93.98 0)
+      (effects (font (size 1.27 1.27)) hide)
+    )
+    (pin "1")
+    (pin "2")
+    (instances
+      (project "Weather Station Motherboard V1"
+        (path "/782b25c2-8b22-49ba-9398-f7481b8d9716"
+          (reference "JP3") (unit 1)
+        )
+      )
+    )
+  )
   (symbol (lib_id "Device:R") (at 72.39 160.02 90) (unit 1)
     (in_bom yes) (on_board yes) (dnp no)
@@
         )
       )
+    )
+  )
+  (symbol (lib_id "Jumper:SolderJumper_2_Open") (at 190.5 115.57 0) (unit 1)
+    (in_bom yes) (on_board yes) (dnp no) (fields_autoplaced)
+    (property "Reference" "JP1" (at 190.5 109.22 0)
+      (effects (font (size 1.27 1.27)))
+    )
+    (property "Value" "SolderJumper_2_Open" (at 190.5 111.76 0)
+      (effects (font (size 1.27 1.27)))
+    )
+    (property "Footprint" "Jumper:SolderJumper-2_P1.3mm_Open_RoundedPad1.0x1.5mm" (at 190.5 115.57 0)
+      (effects (font (size 1.27 1.27)) hide)
+    )
+    (property "Datasheet" "~" (at 190.5 115.57 0)
+      (effects (font (size 1.27 1.27)) hide)
+    )
+    (pin "1")
+    (pin "2")
+    (instances
+      (project "Weather Station Motherboard V1"
+        (path "/782b25c2-8b22-49ba-9398-f7481b8d9716"
+          (reference "JP1") (unit 1)
+        )
+      )
