File: hardware/Weather Station Motherboard V1/Weather Station Motherboard V1.kicad_sch (KiCad schematic)
At the start: 37 parts, among them J1 Conn_01x02, J2 Conn_02x03_Odd_Even, J3 Conn_01x04, U1 ESP32-WROOM-32, U2 SHTC3, U3 BMP390, U4 TPS62177DQC

Commit message: On Board Pressure Sensors
Rerouted on board pressure sensors for SPI with solderable breaks in connections. Added telemetry unit.
Parts:
- added C10, C6, C7: 100n, symbol Device:C
- added H1, H2, H3, H4: MountingHole, symbol Mechanical:MountingHole
- added JP10, JP5, JP6, JP7, JP8, JP9: SolderJumper_2_Open, Jumper:SolderJumper-2_P1.3mm_Open_RoundedPad1.0x1.5mm, symbol Jumper:SolderJumper_2_Open
- added R13, R14, R6: 10k, symbol Device:R
- added U9: NRF24L01_Breakout, RF_Module:nRF24L01_Breakout, symbol RF:NRF24L01_Breakout
Connections:
- net +3.3V: now also U5.9 (VDD), U6.9 (VDD), U7.9 (VDD), C10.1, C6.1, C7.1, R13.2, R14.2, R6.2, U9.2 (VCC)
- net GND: now also U5.8 (Gnd), U6.8 (Gnd), U7.8 (Gnd), C10.2, C6.2, C7.2, U9.1 (GND)
- net nSS_{3}_S: now reaches U7.1 (nSS)
- net nSS_{3}_S: now also JP7.1 (A)
- net nRST_S: now reaches U7.10 (nRST)
- net nRST_S: now also JP1.1 (A), U5.10 (nRST), U6.10 (nRST)
- net DAV_{3}_S: now reaches U7.11 (DAV)
- net DAV_{3}_S: now also JP10.1 (A)
- net MOSI_S: now reaches U7.2 (MOSI)
- net MOSI_S: now also JP3.1 (A), U5.2 (MOSI), U6.2 (MOSI)
- net MISO_S: now reaches U7.3 (MISO)
- net MISO_S: now also JP4.1 (A), U5.3 (MISO), U6.3 (MISO)
- net SCK_S: now reaches U7.4 (SCK)
- net SCK_S: now also JP2.1 (A), U5.4 (SCK), U6.4 (SCK)
- net MISO: now reaches JP4.2 (B)
- net MISO: now also U1.31 (IO19), U9.7 (MISO)
- net nSS_{1}_S: now reaches U5.1 (nSS)
- net nSS_{1}_S: now also JP5.1 (A)
- net DAV_{1}_S: now reaches U5.11 (DAV)
- net DAV_{1}_S: now also JP8.1 (A)
- net SCK: now reaches JP2.2 (B)
- net SCK: now also U1.30 (IO18), U9.5 (SCK)
- net nSS_{2}_S: now reaches U6.1 (nSS)
- net nSS_{2}_S: now also JP6.1 (A)
- net DAV_{2}_S: now reaches U6.11 (DAV)
- net DAV_{2}_S: now also JP9.1 (A)
- net nRST: now reaches U1.10 (IO25)
- net nRST: now also JP1.2 (B)
- net nSS_{1}: now reaches U1.11 (IO26)
- net nSS_{1}: now also JP5.2 (B), R14.1
- net nSS_{2}: now reaches U1.12 (IO27)
- net nSS_{2}: now also JP6.2 (B), R13.1
- net RF_{SEL}: now reaches U1.24 (IO2)
- net RF_{SEL}: now also U9.4 (~{CSN})
- net RF_{EN}: now reaches U1.26 (IO4)
- net RF_{EN}: now also U9.3 (CE)
- net RF_{INT}: now reaches U1.29 (IO5)
- net RF_{INT}: now also U9.8 (IRQ)
- net MOSI: now reaches U1.37 (IO23)
- net MOSI: now also JP3.2 (B), U9.6 (MOSI)
- net DAV_{2}: now reaches U1.6 (IO34)
- net DAV_{2}: now also JP9.2 (B)
- net DAV_{3}: now reaches U1.7 (IO35)
- net DAV_{3}: now also JP10.2 (B)
- net nSS_{3}: now reaches U1.8 (IO32)
- net nSS_{3}: now also JP7.2 (B), R6.1
- net DAV_{1}: now reaches U1.9 (IO33)
- net DAV_{1}: now also JP8.2 (B)
- no-connect marks 24 -> 11
Other:
- moved on the sheet: C1, C2, C3, J2, J3, JP1, JP2, JP3, JP4, R1, R2, R3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
