File: hardware/motherboard/motherboard.kicad_sch (KiCad schematic)
At the start: 56 parts, among them J1 Conn_01x02, J2 Conn_02x03_Odd_Even, J3 Conn_01x04, U1 ESP32-WROOM-32, U2 SHTC3, U3 BMP390, U4 TPS62177DQC, U8 NRF24L01_Breakout

Commit message: Initial PCB design
Initial PCB design complete
Parts:
- removed R5: 100k, Resistor_SMD:R_0603_1608Metric, symbol Device:R
Connections:
- net GND: no longer C10.2, C6.2, C7.2
- net GND1: now also C10.2, C6.2, C7.2
- no-connect marks 11 -> 12
Changed lines of the file:
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@@
   (junction (at 57.15 27.94) (diameter 0) (color 0 0 0 0)
   )
-  (junction (at 127 160.02) (diameter 0) (color 0 0 0 0)
-  )
   (junction (at 147.32 40.64) (diameter 0) (color 0 0 0 0)
   )
@@
   (no_connect (at 189.23 45.72))
   (no_connect (at 27.94 48.26))
+  (no_connect (at 90.17 172.72))
   (no_connect (at 27.94 78.74))
   (wire (pts (xy 121.92 93.98) (xy 140.97 93.98))
@@
     (stroke (width 0) (type default))
   )
-  (wire (pts (xy 90.17 172.72) (xy 86.36 172.72))
-    (stroke (width 0) (type default))
-  )
   (wire (pts (xy 33.02 160.02) (xy 39.37 160.02))
     (stroke (width 0) (type default))
@@
     (stroke (width 0) (type default))
   )
-  (wire (pts (xy 86.36 172.72) (xy 86.36 194.31))
-    (stroke (width 0) (type default))
-  )
   (wire (pts (xy 204.47 105.41) (xy 207.01 105.41))
     (stroke (width 0) (type default))
@@
     (stroke (width 0) (type default))
   )
-  (wire (pts (xy 86.36 194.31) (xy 127 194.31))
-    (stroke (width 0) (type default))
-  )
-  (wire (pts (xy 127 167.64) (xy 127 194.31))
-    (stroke (width 0) (type default))
-  )
   (wire (pts (xy 95.25 180.34) (xy 95.25 182.88))
     (stroke (width 0) (type default))
@@
     )
   )
+  (symbol (lib_id "power:GND1") (at 248.92 27.94 90) (unit 1)
+    (in_bom yes) (on_board yes) (dnp no) (fields_autoplaced)
+    (property "Reference" "#PWR034" (at 255.27 27.94 0)
+      (effects (font (size 1.27 1.27)) hide)
+    )
+    (property "Value" "GND1" (at 252.73 27.94 90)
+      (effects (font (size 1.27 1.27)) (justify right))
+    )
+    (property "Footprint" "" (at 248.92 27.94 0)
+      (effects (font (size 1.27 1.27)) hide)
+    )
+    (property "Datasheet" "" (at 248.92 27.94 0)
+      (effects (font (size 1.27 1.27)) hide)
+    )
+    (pin "1")
+    (instances
+      (project "motherboard"
+        (path "/782b25c2-8b22-49ba-9398-f7481b8d9716"
+          (reference "#PWR034") (unit 1)
+        )
+      )
+    )
+  )
   (symbol (lib_id "Jumper:SolderJumper_2_Open") (at 200.66 143.51 180) (unit 1)
     (in_bom yes) (on_board yes) (dnp no)
@@
     )
   )
-  (symbol (lib_id "power:GND") (at 248.92 74.93 90) (unit 1)
-    (in_bom yes) (on_board yes) (dnp no) (fields_autoplaced)
-    (property "Reference" "#PWR033" (at 255.27 74.93 0)
-      (effects (font (size 1.27 1.27)) hide)
-    )
-    (property "Value" "GND" (at 252.73 74.93 90)
-      (effects (font (size 1.27 1.27)) (justify right))
-    )
-    (property "Footprint" "" (at 248.92 74.93 0)
-      (effects (font (size 1.27 1.27)) hide)
-    )
-    (property "Datasheet" "" (at 248.92 74.93 0)
-      (effects (font (size 1.27 1.27)) hide)
-    )
-    (pin "1")
-    (instances
-      (project "motherboard"
-        (path "/782b25c2-8b22-49ba-9398-f7481b8d9716"
-          (reference "#PWR033") (unit 1)
-        )
-      )
-    )
-  )
   (symbol (lib_id "Device:C") (at 193.04 38.1 90) (unit 1)
     (in_bom yes) (on_board yes) (dnp no)
@@
     )
   )
+  (symbol (lib_id "power:GND1") (at 248.92 124.46 90) (unit 1)
+    (in_bom yes) (on_board yes) (dnp no) (fields_autoplaced)
+    (property "Reference" "#PWR021" (at 255.27 124.46 0)
+      (effects (font (size 1.27 1.27)) hide)
+    )
+    (property "Value" "GND1" (at 252.73 124.46 90)
+      (effects (font (size 1.27 1.27)) (justify right))
+    )
+    (property "Footprint" "" (at 248.92 124.46 0)
+      (effects (font (size 1.27 1.27)) hide)
+    )
+    (property "Datasheet" "" (at 248.92 124.46 0)
+      (effects (font (size 1.27 1.27)) hide)
+    )
+    (pin "1")
+    (instances
+      (project "motherboard"
+        (path "/782b25c2-8b22-49ba-9398-f7481b8d9716"
+          (reference "#PWR021") (unit 1)
+        )
+      )
+    )
+  )
   (symbol (lib_id "power:GND1") (at 207.01 86.36 90) (unit 1)
     (in_bom yes) (on_board yes) (dnp no) (fields_autoplaced)
@@
     )
   )
+  (symbol (lib_id "power:GND1") (at 248.92 74.93 90) (unit 1)
+    (in_bom yes) (on_board yes) (dnp no) (fields_autoplaced)
+    (property "Reference" "#PWR031" (at 255.27 74.93 0)
+      (effects (font (size 1.27 1.27)) hide)
+    )
+    (property "Value" "GND1" (at 252.73 74.93 90)
+      (effects (font (size 1.27 1.27)) (justify right))
+    )
+    (property "Footprint" "" (at 248.92 74.93 0)
+      (effects (font (size 1.27 1.27)) hide)
+    )
+    (property "Datasheet" "" (at 248.92 74.93 0)
+      (effects (font (size 1.27 1.27)) hide)
+    )
+    (pin "1")
+    (instances
+      (project "motherboard"
+        (path "/782b25c2-8b22-49ba-9398-f7481b8d9716"
+          (reference "#PWR031") (unit 1)
+        )
+      )
+    )
+  )
   (symbol (lib_id "power:GND") (at 93.98 71.12 90) (unit 1)
     (in_bom yes) (on_board yes) (dnp no) (fields_autoplaced)
@@
     )
   )
-  (symbol (lib_id "Device:R") (at 127 163.83 0) (unit 1)
-    (in_bom yes) (on_board yes) (dnp no) (fields_autoplaced)
-    (property "Reference" "R5" (at 129.54 162.56 0)
-      (effects (font (size 1.27 1.27)) (justify left))
-    )
-    (property "Value" "100k" (at 129.54 165.1 0)
-      (effects (font (size 1.27 1.27)) (justify left))
-    )
-    (property "Footprint" "Resistor_SMD:R_0603_1608Metric" (at 125.222 163.83 90)
-      (effects (font (size 1.27 1.27)) hide)
-    )
-    (property "Datasheet" "~" (at 127 163.83 0)
-      (effects (font (size 1.27 1.27)) hide)
-    )
-    (pin "1")
-    (pin "2")
-    (instances
-      (project "motherboard"
-        (path "/782b25c2-8b22-49ba-9398-f7481b8d9716"
-          (reference "R5") (unit 1)
-        )
-      )
-    )
-  )
   (symbol (lib_id "RF_Module:ESP32-WROOM-32D") (at 43.18 73.66 0) (unit 1)
     (in_bom yes) (on_board yes) (dnp no)
@@
     )
   )
-  (symbol (lib_id "power:GND") (at 248.92 124.46 90) (unit 1)
-    (in_bom yes) (on_board yes) (dnp no) (fields_autoplaced)
-    (property "Reference" "#PWR036" (at 255.27 124.46 0)
-      (effects (font (size 1.27 1.27)) hide)
-    )
-    (property "Value" "GND" (at 252.73 124.46 90)
-      (effects (font (size 1.27 1.27)) (justify right))
-    )
-    (property "Footprint" "" (at 248.92 124.46 0)
-      (effects (font (size 1.27 1.27)) hide)
-    )
-    (property "Datasheet" "" (at 248.92 124.46 0)
-      (effects (font (size 1.27 1.27)) hide)
-    )
-    (pin "1")
-    (instances
-      (project "motherboard"
-        (path "/782b25c2-8b22-49ba-9398-f7481b8d9716"
-          (reference "#PWR036") (unit 1)
-        )
-      )
-    )
-  )
   (symbol (lib_id "Device:LED") (at 74.93 71.12 180) (unit 1)
     (in_bom yes) (on_board yes) (dnp no)
@@
         )
       )
-    )
-  )
-  (symbol (lib_id "power:GND") (at 248.92 27.94 90) (unit 1)
-    (in_bom yes) (on_board yes) (dnp no) (fields_autoplaced)
-    (property "Reference" "#PWR030" (at 255.27 27.94 0)
-      (effects (font (size 1.27 1.27)) hide)
-    )
-    (property "Value" "GND" (at 252.73 27.94 90)
-      (effects (font (size 1.27 1.27)) (justify right))
-    )
-    (property "Footprint" "" (at 248.92 27.94 0)
-      (effects (font (size 1.27 1.27)) hide)
-    )
-    (property "Datasheet" "" (at 248.92 27.94 0)
-      (effects (font (size 1.27 1.27)) hide)
-    )
-    (pin "1")
-    (instances
-      (project "motherboard"
-        (path "/782b25c2-8b22-49ba-9398-f7481b8d9716"
-          (reference "#PWR030") (unit 1)
-        )
-      )

Commit message: Hole change
Parts:
- H1, H2, H3, H4, JP1, JP10, JP11, JP12, JP2, JP3, JP4, JP5, JP6, JP7, JP8, JP9: now left out of the parts list
Changed lines of the file:
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@@
   )
   (symbol (lib_id "Jumper:SolderJumper_2_Open") (at 200.66 143.51 180) (unit 1)
-    (in_bom yes) (on_board yes) (dnp no)
+    (in_bom no) (on_board yes) (dnp no)
     (property "Reference" "JP9" (at 205.74 142.24 0)
       (effects (font (size 1.27 1.27)) (justify left))
@@
   )
   (symbol (lib_id "Jumper:SolderJumper_2_Open") (at 200.66 149.86 180) (unit 1)
-    (in_bom yes) (on_board yes) (dnp no)
+    (in_bom no) (on_board yes) (dnp no)
     (property "Reference" "JP10" (at 207.01 148.59 0)
       (effects (font (size 1.27 1.27)) (justify left))
@@
   )
   (symbol (lib_id "Jumper:SolderJumper_2_Open") (at 200.66 80.01 180) (unit 1)
-    (in_bom yes) (on_board yes) (dnp no)
+    (in_bom no) (on_board yes) (dnp no)
     (property "Reference" "JP12" (at 207.01 78.74 0)
       (effects (font (size 1.27 1.27)) (justify left))
@@
   )
   (symbol (lib_id "Jumper:SolderJumper_2_Open") (at 200.66 111.76 180) (unit 1)
-    (in_bom yes) (on_board yes) (dnp no)
+    (in_bom no) (on_board yes) (dnp no)
     (property "Reference" "JP4" (at 205.74 110.49 0)
       (effects (font (size 1.27 1.27)) (justify left))
@@
   )
   (symbol (lib_id "Jumper:SolderJumper_2_Open") (at 200.66 118.11 180) (unit 1)
-    (in_bom yes) (on_board yes) (dnp no)
+    (in_bom no) (on_board yes) (dnp no)
     (property "Reference" "JP5" (at 205.74 116.84 0)
       (effects (font (size 1.27 1.27)) (justify left))
@@
   )
   (symbol (lib_id "Jumper:SolderJumper_2_Open") (at 200.66 124.46 180) (unit 1)
-    (in_bom yes) (on_board yes) (dnp no)
+    (in_bom no) (on_board yes) (dnp no)
     (property "Reference" "JP6" (at 205.74 123.19 0)
       (effects (font (size 1.27 1.27)) (justify left))
@@
   )
   (symbol (lib_id "Jumper:SolderJumper_2_Open") (at 200.66 86.36 180) (unit 1)
-    (in_bom yes) (on_board yes) (dnp no)
+    (in_bom no) (on_board yes) (dnp no)
     (property "Reference" "JP11" (at 207.01 85.09 0)
       (effects (font (size 1.27 1.27)) (justify left))
@@
   )
   (symbol (lib_id "Mechanical:MountingHole") (at 284.48 24.13 0) (unit 1)
-    (in_bom yes) (on_board yes) (dnp no) (fields_autoplaced)
+    (in_bom no) (on_board yes) (dnp no) (fields_autoplaced)
     (property "Reference" "H1" (at 287.02 22.86 0)
       (effects (font (size 1.27 1.27)) (justify left))
@@
   )
   (symbol (lib_id "Jumper:SolderJumper_2_Open") (at 200.66 92.71 180) (unit 1)
-    (in_bom yes) (on_board yes) (dnp no)
+    (in_bom no) (on_board yes) (dnp no)
     (property "Reference" "JP1" (at 205.74 91.44 0)
       (effects (font (size 1.27 1.27)) (justify left))
@@
   )
   (symbol (lib_id "Jumper:SolderJumper_2_Open") (at 200.66 137.16 180) (unit 1)
-    (in_bom yes) (on_board yes) (dnp no)
+    (in_bom no) (on_board yes) (dnp no)
     (property "Reference" "JP8" (at 205.74 135.89 0)
       (effects (font (size 1.27 1.27)) (justify left))
@@
   )
   (symbol (lib_id "Mechanical:MountingHole") (at 284.48 36.83 0) (unit 1)
-    (in_bom yes) (on_board yes) (dnp no) (fields_autoplaced)
+    (in_bom no) (on_board yes) (dnp no) (fields_autoplaced)
     (property "Reference" "H3" (at 287.02 35.56 0)
       (effects (font (size 1.27 1.27)) (justify left))
@@
   )
   (symbol (lib_id "Jumper:SolderJumper_2_Open") (at 200.66 105.41 180) (unit 1)
-    (in_bom yes) (on_board yes) (dnp no)
+    (in_bom no) (on_board yes) (dnp no)
     (property "Reference" "JP3" (at 205.74 104.14 0)
       (effects (font (size 1.27 1.27)) (justify left))
@@
   )
   (symbol (lib_id "Mechanical:MountingHole") (at 284.48 43.18 0) (unit 1)
-    (in_bom yes) (on_board yes) (dnp no) (fields_autoplaced)
+    (in_bom no) (on_board yes) (dnp no) (fields_autoplaced)
     (property "Reference" "H4" (at 287.02 41.91 0)
       (effects (font (size 1.27 1.27)) (justify left))
@@
   )
   (symbol (lib_id "Jumper:SolderJumper_2_Open") (at 200.66 99.06 180) (unit 1)
-    (in_bom yes) (on_board yes) (dnp no)
+    (in_bom no) (on_board yes) (dnp no)
     (property "Reference" "JP2" (at 205.74 97.79 0)
       (effects (font (size 1.27 1.27)) (justify left))
@@
   )
   (symbol (lib_id "Jumper:SolderJumper_2_Open") (at 200.66 130.81 180) (unit 1)
-    (in_bom yes) (on_board yes) (dnp no)
+    (in_bom no) (on_board yes) (dnp no)
     (property "Reference" "JP7" (at 205.74 129.54 0)
       (effects (font (size 1.27 1.27)) (justify left))
@@
   )
   (symbol (lib_id "Mechanical:MountingHole") (at 284.48 30.48 0) (unit 1)
-    (in_bom yes) (on_board yes) (dnp no) (fields_autoplaced)
+    (in_bom no) (on_board yes) (dnp no) (fields_autoplaced)
     (property "Reference" "H2" (at 287.02 29.21 0)
       (effects (font (size 1.27 1.27)) (justify left))
